File: schema/mjBeep/boardBase2.brd (EAGLE design)
At the start: 100 x 62.2 mm, 18 parts, among them IC1 atmega1284, Q1 16MH, T1 BC547, X2 VIN

Commit message: mod
Parts:
- added IC2, IC3: PCF8574P, micro-philips:DIL16
- added JP3, JP5, JP7: (no value), pinhead:2X03
- added KEYPAD: (no value), pinhead:1X08
- added LED1: (no value), led:LED3MM
- added R10, R11, R12, R13, R14, R15, R6, R7, R8, R9: 10K, rcl:0207/10
- added R16, R17: 220, rcl:0207/10
- JP1: value LedPin -> (none); device pinhead:2X03 -> pinhead:1X05
- moved JP2 71.4 mm to (22.9, 38.1), turned to 0 degrees
- moved JP4 63.6 mm to (30.5, 38.1), turned to 0 degrees
- moved C5 56.8 mm to (63.5, 48.3)
- moved X2 55.8 mm to (68.6, 30.5), turned to 0 degrees
- moved T1 52.6 mm to (47.0, 54.6), turned to 0 degrees
- moved SV1 51.2 mm to (64.8, 54.6)
- moved R5 48.5 mm to (41.9, 59.7), turned to 0 degrees
- moved R3 45.8 mm to (67.3, 59.7), turned to 0 degrees
- moved C3 39.1 mm to (16.5, 38.1)
- moved R4 36.9 mm to (54.6, 59.7), turned to 0 degrees
- moved JP1 35.9 mm to (21.6, 47.0)
- moved C2 34.5 mm to (52.1, 48.3), turned to 0 degrees
- moved IC1 31.4 mm to (47.0, 11.4)
- moved R2 27.7 mm to (25.4, 53.3), turned to 0 degrees
- moved R1 27.2 mm to (38.1, 53.3)
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Connections:
- new net LED_SIRENA: IC1.5, R16.1
- new net N$10: IC2.14, R10.1
- new net N$13: IC2.15, R9.1
- new net N$14: IC3.1, JP7.2, R13.2
- new net N$15: IC3.2, JP7.4, R11.2
- new net N$16: IC3.3, JP7.6, R12.1
- new net N$17: IC3.14, R15.1
- new net N$18: IC3.15, R14.1
- new net N$19: JP1.5, R16.2
- new net N$20: IC1.1, R17.1
- new net N$21: LED1.A, R17.2
- new net N$3: IC2.1, JP3.2, R8.2
- new net N$5: IC2.2, JP3.4, R6.2
- new net N$6: IC2.3, JP3.6, R7.1
- new net P0: IC2.4, KEYPAD.5
- new net P1: IC2.5, KEYPAD.6
- new net P2: IC2.6, KEYPAD.7
- new net P3: IC2.7, KEYPAD.8
- new net P4: IC2.9, KEYPAD.1
- new net P5: IC2.10, KEYPAD.2
- new net P6: IC2.11, KEYPAD.3
- new net P7: IC2.12, KEYPAD.4
- new net SCL: IC1.22, R10.2, R15.2
- new net SDA: IC1.23, R14.2, R9.2
- net 5V: now also IC2.16, IC3.16, R11.1, R12.2, R13.1, R6.1, R7.2, R8.1
- net GND: now also IC2.8, IC3.8, JP3.1, JP3.3, JP3.5, JP7.1, JP7.3, JP7.5, LED1.K; no longer JP1.3, JP1.5
- net N$7: now also JP1.4; no longer JP1.2
- net N$8: now also JP1.3; no longer JP1.4
- net N$9: now also JP1.2; no longer JP1.6
Other:
- board size 100 x 62.2 mm -> 100 x 80 mm
