File: schema/mjBeep/boardBase2.sch (EAGLE design)
At the start: 18 parts, among them IC1 atmega1284, Q1 16MH, T1 BC547, X2 VIN

Commit message: mod
Parts:
- added IC2, IC3: PCF8574P, micro-philips:PCF8574P
- added JP3, JP5, JP7: (no value), pinhead:PINHD-2X3
- added KEYPAD: (no value), pinhead:PINHD-1X8
- added LED1: (no value), led:LED3MM
- added R10, R11, R12, R13, R14, R15, R6, R7, R8, R9: 10K, rcl:R-EU_0207/10
- added R16, R17: 220, rcl:R-EU_0207/10
- JP1: value LedPin -> (none); device pinhead:PINHD-2X3 -> pinhead:PINHD-1X5
Connections:
- new net LED_SIRENA: IC1.SS/OC0B/PCINT12, R16.1
- new net N$10: IC2.SCL, R10.1
- new net N$13: IC2.SDA, R9.1
- new net N$14: IC3.A0, JP7.2, R13.2
- new net N$15: IC3.A1, JP7.4, R11.2
- new net N$16: IC3.A2, JP7.6, R12.1
- new net N$17: IC3.SCL, R15.1
- new net N$18: IC3.SDA, R14.1
- new net N$19: JP1.5, R16.2
- new net N$20: IC1.T0/XCK0/PCINT8, R17.1
- new net N$21: LED1.A, R17.2
- new net N$3: IC2.A0, JP3.2, R8.2
- new net N$5: IC2.A1, JP3.4, R6.2
- new net N$6: IC2.A2, JP3.6, R7.1
- new net P0: IC2.P0, KEYPAD.5
- new net P1: IC2.P1, KEYPAD.6
- new net P2: IC2.P2, KEYPAD.7
- new net P3: IC2.P3, KEYPAD.8
- new net P4: IC2.P4, KEYPAD.1
- new net P5: IC2.P5, KEYPAD.2
- new net P6: IC2.P6, KEYPAD.3
- new net P7: IC2.P7, KEYPAD.4
- new net SCL: IC1.SCL/PCINT16, R10.2, R15.2
- new net SDA: IC1.SDA/PCINT17, R14.2, R9.2
- net 5V: now also IC2.VDD, IC3.VDD, R11.1, R12.2, R13.1, R6.1, R7.2, R8.1
- net GND: now also IC2.VSS, IC3.VSS, JP3.1, JP3.3, JP3.5, JP7.1, JP7.3, JP7.5, LED1.C; no longer JP1.3, JP1.5
- net N$7: now also JP1.4; no longer JP1.2
- net N$8: now also JP1.3; no longer JP1.4
- net N$9: now also JP1.2; no longer JP1.6
Other:
- note added: "KeyPAD"
- moved on the sheet: C5, JP2, JP4, R2, R3, R4, R5, SV1, T1, X2-1, X2-2

Commit message: mod
Parts:
- added JP8: (no value), pinhead:PINHD-1X16
- added R18, R19, R20, R21, R22, R23, R24, R25: 10K, rcl:R-EU_0207/10
- added S1: (no value), switch-omron:10-XX
- added X1, X3: (no value), con-wago-508:W237-08P
Connections:
- new net N$22: IC3.P0, JP8.2, X1-8.KL
- new net N$23: IC3.P1, JP8.4, X1-6.KL
- new net N$24: IC3.P2, JP8.6, X1-4.KL
- new net N$25: IC3.P3, JP8.8, X1-2.KL
- new net N$26: IC3.P4, JP8.10, X3-8.KL
- new net N$27: IC3.P5, JP8.12, X3-6.KL
- new net N$28: IC3.P6, JP8.14, X3-4.KL
- new net N$29: IC3.P7, JP8.16, X3-2.KL
- new net N$30: JP8.1, R18.2
- new net N$31: JP8.3, R19.2
- new net N$32: JP8.5, R20.2
- new net N$33: JP8.7, R21.2
- new net N$34: JP8.9, R22.2
- new net N$35: JP8.11, R23.2
- new net N$36: JP8.13, R24.2
- new net N$37: JP8.15, R25.2
- new net N$40: R20.1
- net 5V: now also X1-1.KL, X1-3.KL, X1-5.KL, X1-7.KL, X3-1.KL, X3-3.KL, X3-5.KL, X3-7.KL
- net GND: now also R18.1, R19.1, R21.1, R22.1, R23.1, R24.1, R25.1, S1.S
- net RESET: now also S1.P
Other:
- note added: "5V"
- note added: "GND"

Commit message: mod
Other:
- note added: "RTC"
Changed lines of the file:
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@@
 <?xml version="1.0" encoding="utf-8"?>
 <!DOCTYPE eagle SYSTEM "eagle.dtd">
-<eagle version="8.3.2">
+<eagle version="8.4.0">
 <drawing>
 <settings>
@@
 <text x="246.38" y="-40.64" size="1.778" layer="91">5V</text>
 <text x="246.38" y="-50.8" size="1.778" layer="91">5V</text>
+<text x="-5.08" y="-25.4" size="1.778" layer="91">RTC</text>
 </plain>
 <instances>
