File: schema/mjBeep/alimentazione.brd (EAGLE design)
At the start: 105.1 x 85.1 mm, 19 parts, among them IC1 LM317, IC2 LM317, IC3 7805T, J1 Alimentazione, J2 BATTERIA, J3 OUT, T1 BC547

Commit message: mod
Parts:
- IC2: value LM317 -> LM350
- moved J3 48.0 mm to (67.3, 66.0), turned to 270 degrees
- moved IC3 45.4 mm to (39.4, 43.2), turned to 90 degrees
- moved C1 33.6 mm to (30.5, 59.7), turned to 270 degrees
- moved C3 31.9 mm to (62.2, 35.6)
- moved D3 27.3 mm to (35.6, 66.0)
- moved R6 27.3 mm to (35.6, 71.1)
- moved R7 26.7 mm to (52.1, 63.5), turned to 0 degrees
- moved D4 24.3 mm to (50.8, 29.2)
- moved R5 21.1 mm to (49.5, 16.5), turned to 270 degrees
- moved C4 19.4 mm to (63.5, 45.7), turned to 180 degrees
- moved T1 18.1 mm to (29.2, 5.08)
- moved R3 17.0 mm to (41.9, 6.35)
- moved J2 16.9 mm to (64.8, 17.8), turned to 270 degrees
- moved IC1 10.9 mm to (17.8, 20.3)
- moved J1 9.67 mm to (8.89, 40.6), turned to 90 degrees
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Connections:
- net N$6 renamed 5V
Other:
- board size 105.1 x 85.1 mm -> 81 x 80 mm

Commit message: mod
Parts:
- added J4: OUT, Libreria-componenti:MORSETTIERA
- moved C4 6.35 mm to (59.7, 50.8), turned to 270 degrees
- moved C3 6.35 mm to (58.4, 40.6), turned to 90 degrees
Connections:
- removed net N$9: C3.+, D3.C, D4.C, IC3.1
- new net 13.8V: C3.+, D3.C, D4.C, IC3.1, J4.1
- net GND: now also J4.2
Changed lines of the file:
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@@
 </autorouter>
 <elements>
-<element name="C3" library="rcl" package="E2,5-6" value="100nF" x="62.23" y="35.56"/>
-<element name="C4" library="rcl" package="E2,5-6" value="100nF" x="63.5" y="45.72" rot="R180"/>
+<element name="C3" library="rcl" package="E2,5-6" value="100nF" x="58.42" y="40.64" rot="R90"/>
+<element name="C4" library="rcl" package="E2,5-6" value="100nF" x="59.69" y="50.8" rot="R270"/>
 <element name="D1" library="Libreria-componenti" package="DO41-10" value="1N4001" x="31.75" y="22.86" rot="R180"/>
 <element name="D3" library="Libreria-componenti" package="DO41-10" value="1N4001" x="35.56" y="66.04" rot="R180"/>
@@
 <element name="T1" library="transistor-npn" package="TO92" value="BC547" x="29.21" y="5.08" rot="R270"/>
 <element name="C1" library="rcl" package="E2,5-6" value="10uF" x="30.48" y="59.69" rot="R270"/>
+<element name="J4" library="Libreria-componenti" package="MORSETTIERA" value="OUT" x="69.85" y="53.34" rot="R270"/>
 </elements>
 <signals>
@@
 <contactref element="C4" pad="-"/>
 <contactref element="C1" pad="-"/>
-<wire x1="49.53" y1="43.18" x2="30.48" y2="58.42" width="0" layer="19" extent="1-1"/>
-<wire x1="67.31" y1="60.96" x2="49.53" y2="43.18" width="0" layer="19" extent="1-1"/>
-<wire x1="63.5" y1="35.56" x2="67.31" y2="60.96" width="0" layer="19" extent="1-1"/>
-<wire x1="8.89" y1="45.72" x2="67.31" y2="60.96" width="0" layer="19" extent="1-1"/>
-<wire x1="49.53" y1="58.42" x2="8.89" y2="45.72" width="0" layer="19" extent="1-1"/>
+<contactref element="J4" pad="2"/>
+<wire x1="59.69" y1="49.53" x2="67.31" y2="60.96" width="0" layer="19" extent="1-1"/>
+<wire x1="58.42" y1="41.91" x2="59.69" y2="49.53" width="0" layer="19" extent="1-1"/>
+<wire x1="49.53" y1="43.18" x2="59.69" y2="49.53" width="0" layer="19" extent="1-1"/>
+<wire x1="49.53" y1="58.42" x2="49.53" y2="43.18" width="0" layer="19" extent="1-1"/>
 <wire x1="52.07" y1="68.58" x2="49.53" y2="58.42" width="0" layer="19" extent="1-1"/>
-<wire x1="62.23" y1="45.72" x2="52.07" y2="68.58" width="0" layer="19" extent="1-1"/>
-<wire x1="36.83" y1="2.54" x2="62.23" y2="45.72" width="0" layer="19" extent="1-1"/>
+<wire x1="30.48" y1="58.42" x2="49.53" y2="58.42" width="0" layer="19" extent="1-1"/>
+<wire x1="8.89" y1="45.72" x2="30.48" y2="58.42" width="0" layer="19" extent="1-1"/>
+<wire x1="36.83" y1="2.54" x2="58.42" y2="41.91" width="0" layer="19" extent="1-1"/>
 <wire x1="29.21" y1="3.81" x2="36.83" y2="2.54" width="0" layer="19" extent="1-1"/>
+<wire x1="69.85" y1="48.26" x2="29.21" y2="3.81" width="0" layer="19" extent="1-1"/>
 </signal>
 <signal name="-BAT">
@@
 <wire x1="21.59" y1="62.23" x2="54.61" y2="58.42" width="0" layer="19" extent="1-1"/>
 </signal>
-<signal name="N$9">
+<signal name="13.8V">
 <contactref element="D3" pad="C"/>
 <contactref element="D4" pad="C"/>
 <contactref element="IC3" pad="1"/>
 <contactref element="C3" pad="+"/>
-<wire x1="55.88" y1="29.21" x2="49.53" y2="40.64" width="0" layer="19" extent="1-1"/>
-<wire x1="60.96" y1="35.56" x2="55.88" y2="29.21" width="0" layer="19" extent="1-1"/>
-<wire x1="40.64" y1="66.04" x2="55.88" y2="29.21" width="0" layer="19" extent="1-1"/>
+<contactref element="J4" pad="1"/>
+<wire x1="49.53" y1="40.64" x2="40.64" y2="66.04" width="0" layer="19" extent="1-1"/>
+<wire x1="58.42" y1="39.37" x2="49.53" y2="40.64" width="0" layer="19" extent="1-1"/>
+<wire x1="55.88" y1="29.21" x2="58.42" y2="39.37" width="0" layer="19" extent="1-1"/>
+<wire x1="69.85" y1="53.34" x2="49.53" y2="40.64" width="0" layer="19" extent="1-1"/>
 </signal>
 <signal name="5V">
@@
 <contactref element="J3" pad="1"/>
 <contactref element="C4" pad="+"/>
-<wire x1="67.31" y1="66.04" x2="64.77" y2="45.72" width="0" layer="19" extent="1-1"/>
+<wire x1="67.31" y1="66.04" x2="59.69" y2="52.07" width="0" layer="19" extent="1-1"/>
 <wire x1="49.53" y1="45.72" x2="67.31" y2="66.04" width="0" layer="19" extent="1-1"/>
 </signal>

Commit message: mod
Parts:
- moved J4 15.3 mm to (68.6, 38.1)
- moved IC3 4.02 mm to (35.6, 41.9)
Changed lines of the file:
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@@
 <?xml version="1.0" encoding="utf-8"?>
 <!DOCTYPE eagle SYSTEM "eagle.dtd">
-<eagle version="7.5.0">
+<eagle version="7.7.0">
 <drawing>
 <settings>
@@
 <element name="IC1" library="v-reg" package="317TL" value="LM317" x="17.78" y="20.32" rot="R90"/>
 <element name="IC2" library="v-reg" package="317TL" value="LM350" x="17.78" y="64.77" rot="R90"/>
-<element name="IC3" library="linear" package="TO220H" value="7805T" x="39.37" y="43.18" rot="R90"/>
+<element name="IC3" library="linear" package="TO220H" value="7805T" x="35.56" y="41.91" rot="R90"/>
 <element name="J1" library="Libreria-componenti" package="MORSETTIERA" value="Alimentazione" x="8.89" y="40.64" rot="R90"/>
 <element name="J2" library="Libreria-componenti" package="MORSETTIERA" value="BATTERIA" x="64.77" y="17.78" rot="R270"/>
@@
 <element name="T1" library="transistor-npn" package="TO92" value="BC547" x="29.21" y="5.08" rot="R270"/>
 <element name="C1" library="rcl" package="E2,5-6" value="10uF" x="30.48" y="59.69" rot="R270"/>
-<element name="J4" library="Libreria-componenti" package="MORSETTIERA" value="OUT" x="69.85" y="53.34" rot="R270"/>
+<element name="J4" library="Libreria-componenti" package="MORSETTIERA" value="OUT" x="68.58" y="38.1" rot="R270"/>
 </elements>
 <signals>
@@
 <wire x1="59.69" y1="49.53" x2="67.31" y2="60.96" width="0" layer="19" extent="1-1"/>
 <wire x1="58.42" y1="41.91" x2="59.69" y2="49.53" width="0" layer="19" extent="1-1"/>
-<wire x1="49.53" y1="43.18" x2="59.69" y2="49.53" width="0" layer="19" extent="1-1"/>
-<wire x1="49.53" y1="58.42" x2="49.53" y2="43.18" width="0" layer="19" extent="1-1"/>
+<wire x1="45.72" y1="41.91" x2="59.69" y2="49.53" width="0" layer="19" extent="1-1"/>
+<wire x1="49.53" y1="58.42" x2="45.72" y2="41.91" width="0" layer="19" extent="1-1"/>
 <wire x1="52.07" y1="68.58" x2="49.53" y2="58.42" width="0" layer="19" extent="1-1"/>
 <wire x1="30.48" y1="58.42" x2="49.53" y2="58.42" width="0" layer="19" extent="1-1"/>
@@
 <wire x1="36.83" y1="2.54" x2="58.42" y2="41.91" width="0" layer="19" extent="1-1"/>
 <wire x1="29.21" y1="3.81" x2="36.83" y2="2.54" width="0" layer="19" extent="1-1"/>
-<wire x1="69.85" y1="48.26" x2="29.21" y2="3.81" width="0" layer="19" extent="1-1"/>
+<wire x1="68.58" y1="33.02" x2="29.21" y2="3.81" width="0" layer="19" extent="1-1"/>
 </signal>
 <signal name="-BAT">
@@
 <contactref element="C3" pad="+"/>
 <contactref element="J4" pad="1"/>
-<wire x1="49.53" y1="40.64" x2="40.64" y2="66.04" width="0" layer="19" extent="1-1"/>
-<wire x1="58.42" y1="39.37" x2="49.53" y2="40.64" width="0" layer="19" extent="1-1"/>
+<wire x1="45.72" y1="39.37" x2="40.64" y2="66.04" width="0" layer="19" extent="1-1"/>
+<wire x1="58.42" y1="39.37" x2="45.72" y2="39.37" width="0" layer="19" extent="1-1"/>
 <wire x1="55.88" y1="29.21" x2="58.42" y2="39.37" width="0" layer="19" extent="1-1"/>
-<wire x1="69.85" y1="53.34" x2="49.53" y2="40.64" width="0" layer="19" extent="1-1"/>
+<wire x1="68.58" y1="38.1" x2="45.72" y2="39.37" width="0" layer="19" extent="1-1"/>
 </signal>
 <signal name="5V">
@@
 <contactref element="C4" pad="+"/>
 <wire x1="67.31" y1="66.04" x2="59.69" y2="52.07" width="0" layer="19" extent="1-1"/>
-<wire x1="49.53" y1="45.72" x2="67.31" y2="66.04" width="0" layer="19" extent="1-1"/>
+<wire x1="45.72" y1="44.45" x2="67.31" y2="66.04" width="0" layer="19" extent="1-1"/>
 </signal>
 </signals>

Commit message: mod
Parts:
- removed IC3: 7805T, linear:TO220H
- added IC4: 7805TV, linear:TO220V
- added U$1, U$2, U$3, U$4: (no value), holes:3,0
- IC1, IC2: device v-reg:317TL -> v-reg:317TS
- moved J3 28.5 mm to (43.2, 50.8)
- moved R5 28.5 mm to (22.9, 6.35), turned to 90 degrees
- moved D4 27.7 mm to (24.1, 21.6), turned to 0 degrees
- moved C4 27.4 mm to (34.3, 40.6)
- moved J4 25.4 mm to (43.2, 39.4)
- moved C3 25.3 mm to (34.3, 33.0), turned to 270 degrees
- moved J2 23.9 mm to (43.2, 27.9)
- moved R6 16.6 mm to (26.7, 57.1)
- moved IC1 16.6 mm to (3.81, 11.4)
- moved IC2 16.6 mm to (3.81, 55.9)
- moved R7 16.5 mm to (35.6, 63.5), turned to 270 degrees
- moved D3 15.5 mm to (26.7, 53.3)
- moved T1 11.4 mm to (34.3, 15.2)
- moved C1 10.2 mm to (21.6, 64.8), turned to 90 degrees
- moved J1 9.25 mm to (6.35, 31.8)
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Connections:
- net 13.8V: now also IC4.1; no longer IC3.1
- net 5V: now also IC4.3; no longer IC3.3
- net GND: now also IC4.2; no longer IC3.2
Routing:
- net GND: track 0.00 -> 173.4 mm
- net 13.8V: track 0.00 -> 65.7 mm
- net -BAT: track 0.00 -> 47.4 mm
- net N$13: track 0.00 -> 46.7 mm
- net N$27: track 0.00 -> 33.5 mm
- net N$5: track 0.00 -> 32.5 mm
- net 5V: track 0.00 -> 27.2 mm
- net N$3: track 0.00 -> 25.4 mm
- net +BAT: track 0.00 -> 20.6 mm
- net N$15: track 0.00 -> 18.2 mm
- net N$4: track 0.00 -> 5.32 mm
- added copper zone on layer 16, net N$1
Other:
- board size 81 x 80 mm -> 55.5 x 87.6 mm
- board text added: "13.8V"
- board text added: "5V"
- board text added: "Bat"
- board text added: "VIN"

Commit message: mod
Parts:
- moved U$1 2.62 mm to (4.45, -1.27)
- moved U$2 2.62 mm to (45.1, -1.27)
- moved U$4 0.64 mm to (4.45, 71.1)
- moved U$3 0.63 mm to (45.1, 71.1)
Routing:
- net GND: track 173.4 -> 120.8 mm
- net 13.8V: track 65.7 -> 58.2 mm
- net N$5: track 32.5 -> 31.4 mm
- removed copper zone on layer 16, net N$1
Other:
- board size 55.5 x 87.6 mm -> 51.7 x 82.5 mm

Commit message: mod
Parts:
- renumbered IC1 to LM317, IC2 to LM350, IC4 to 7805
Changed lines of the file:
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@@
 <setting verticaltext="up"/>
 </settings>
-<grid distance="0.05" unitdist="inch" unit="inch" style="dots" multiple="1" display="yes" altdistance="0.025" altunitdist="inch" altunit="inch"/>
+<grid distance="0.05" unitdist="inch" unit="mm" style="dots" multiple="1" display="yes" altdistance="0.025" altunitdist="inch" altunit="mm"/>
 <layers>
 <layer number="1" name="Top" color="4" fill="1" visible="yes" active="yes"/>
@@
 <attribute name="VALUE" x="49.53" y="41.91" size="1.27" layer="27" rot="R270"/>
 </element>
-<element name="IC1" library="v-reg" library_urn="urn:adsk.eagle:library:409" package="317TS" package3d_urn="urn:adsk.eagle:package:30353/1" value="LM317" x="3.81" y="11.43" smashed="yes" rot="R90">
+<element name="LM317" library="v-reg" library_urn="urn:adsk.eagle:library:409" package="317TS" package3d_urn="urn:adsk.eagle:package:30353/1" value="LM317" x="3.81" y="11.43" smashed="yes" rot="R90">
 <attribute name="NAME" x="9.8552" y="6.35" size="1.27" layer="25" ratio="10" rot="R90"/>
 <attribute name="VALUE" x="11.43" y="6.35" size="1.27" layer="27" ratio="10" rot="R90"/>
 </element>
-<element name="IC2" library="v-reg" library_urn="urn:adsk.eagle:library:409" package="317TS" package3d_urn="urn:adsk.eagle:package:30353/1" value="LM350" x="3.81" y="55.88" smashed="yes" rot="R90">
+<element name="LM350" library="v-reg" library_urn="urn:adsk.eagle:library:409" package="317TS" package3d_urn="urn:adsk.eagle:package:30353/1" value="LM350" x="3.81" y="55.88" smashed="yes" rot="R90">
 <attribute name="NAME" x="9.8552" y="50.8" size="1.27" layer="25" ratio="10" rot="R90"/>
 <attribute name="VALUE" x="11.43" y="50.8" size="1.27" layer="27" ratio="10" rot="R90"/>
 </element>
-<element name="IC4" library="linear" library_urn="urn:adsk.eagle:library:262" package="TO220V" package3d_urn="urn:adsk.eagle:package:16417/1" value="7805TV" x="17.78" y="38.1" smashed="yes" rot="R90">
+<element name="7805" library="linear" library_urn="urn:adsk.eagle:library:262" package="TO220V" package3d_urn="urn:adsk.eagle:package:16417/1" value="7805TV" x="17.78" y="38.1" smashed="yes" rot="R90">
 <attribute name="NAME" x="23.8252" y="33.02" size="1.27" layer="25" ratio="10" rot="R90"/>
 <attribute name="VALUE" x="25.4" y="33.02" size="1.27" layer="27" ratio="10" rot="R90"/>
@@
 <signal name="N$13">
 <contactref element="J1" pad="1"/>
-<contactref element="IC1" pad="3"/>
-<contactref element="IC2" pad="3"/>
+<contactref element="LM317" pad="3"/>
+<contactref element="LM350" pad="3"/>
 <wire x1="6.477" y1="31.5214" x2="6.477" y2="14.2494" width="0.6096" layer="1"/>
 <wire x1="6.477" y1="14.2494" x2="6.35" y2="13.97" width="0.6096" layer="1"/>
@@
 <contactref element="R2" pad="2"/>
 <contactref element="D1" pad="A"/>
-<contactref element="IC1" pad="2"/>
+<contactref element="LM317" pad="2"/>
 <wire x1="16.8402" y1="11.6586" x2="6.477" y2="11.6586" width="0.6096" layer="1"/>
 <wire x1="18.9992" y1="13.8176" x2="16.8402" y2="11.6586" width="0.6096" layer="1"/>
@@
 <contactref element="T1" pad="3"/>
 <contactref element="R5" pad="3"/>
-<contactref element="IC1" pad="1"/>
+<contactref element="LM317" pad="1"/>
 <wire x1="31.5214" y1="16.4084" x2="34.1122" y2="16.4084" width="0.6096" layer="1"/>
 <wire x1="29.3624" y1="14.2494" x2="31.5214" y2="16.4084" width="0.6096" layer="1"/>
@@
 <contactref element="C4" pad="-"/>
 <contactref element="C1" pad="-"/>
-<contactref element="IC4" pad="2"/>
+<contactref element="7805" pad="2"/>
 <contactref element="J4" pad="2"/>
 <contactref element="J3" pad="2"/>
@@
 <contactref element="R6" pad="2"/>
 <contactref element="C1" pad="+"/>
-<contactref element="IC2" pad="2"/>
+<contactref element="LM350" pad="2"/>
 <wire x1="20.7264" y1="56.134" x2="6.477" y2="56.134" width="0.6096" layer="1"/>
 <wire x1="21.59" y1="56.9976" x2="20.7264" y2="56.134" width="0.6096" layer="1"/>
@@
 <contactref element="R7" pad="3"/>
 <contactref element="R6" pad="1"/>
-<contactref element="IC2" pad="1"/>
+<contactref element="LM350" pad="1"/>
 <wire x1="19.431" y1="53.5432" x2="6.477" y2="53.5432" width="0.6096" layer="16"/>
 <wire x1="21.1582" y1="55.2704" x2="19.431" y2="53.5432" width="0.6096" layer="16"/>
@@
 <contactref element="C3" pad="+"/>
 <contactref element="J4" pad="1"/>
-<contactref element="IC4" pad="1"/>
+<contactref element="7805" pad="1"/>
 <wire x1="33.2486" y1="35.4076" x2="31.9532" y2="35.4076" width="0.6096" layer="1"/>
 <wire x1="31.9532" y1="35.4076" x2="20.7264" y2="35.4076" width="0.6096" layer="1"/>
@@
 <contactref element="J3" pad="1"/>
 <contactref element="C4" pad="+"/>
-<contactref element="IC4" pad="3"/>
+<contactref element="7805" pad="3"/>
 <wire x1="33.2486" y1="41.021" x2="20.7264" y2="41.021" width="0.6096" layer="16"/>
 <wire x1="34.1122" y1="41.8846" x2="33.2486" y2="41.021" width="0.6096" layer="16"/>
