File: schema/mjBeep/boardBase.brd (EAGLE design)
At the start: 100 x 80 mm, 17 parts, among them IC1 atmega1284, Q1 16MH, T1 BC547

Commit message: mod
Parts:
- removed LED1, LED2, LED3: (no value), led:LED5MM
- removed X1: (no value), con-wago-500:W237-102
- added C5, C6: 100nF, rcl:E3,5-10
- added IC2: 7805T, linear:TO220H
- added JP1: LedPin, pinhead:2X03
- added JP2: Spk, pinhead:1X02
- added JP3: GSM, pinhead:1X07
- added JP4: Relay, pinhead:1X03
- R5: value (none) -> 230
- X2: value (none) -> VIN
- moved R5 15.5 mm to (76.2, 25.4)
- moved C1 13.1 mm to (66.0, 19.1), turned to 90 degrees
- moved T1 10.8 mm to (76.2, 15.2)
- moved C2 8.89 mm to (57.1, 17.8), turned to 90 degrees
- moved R1 7.41 mm to (43.2, 25.4)
- moved Q1 6.35 mm to (61.0, 25.4)
- moved R4 5.68 mm to (35.6, 25.4)
- moved R3 5.24 mm to (33.0, 25.4)
- moved R2 2.84 mm to (30.5, 25.4)
- moved C4 2.54 mm to (54.6, 53.3)
- moved C3 1.27 mm to (54.6, 29.2)
Connections:
- net N$10 renamed SPK
- removed net N$14: X2.2
- removed net N$4: IC1.1, R2.1
- removed net N$5: IC1.2, R3.1
- removed net N$6: IC1.3, R4.1
- removed net VCC: C3.1, C4.2, IC1.10, IC1.30, R1.1, T1.3
- new net GSM_5V: JP3.7
- new net GSM_GND: JP3.6
- new net LED_GIALLO: IC1.2, R2.1
- new net LED_ROSSO: IC1.4, R4.1
- new net LED_VERDE: IC1.3, R3.1
- new net RELAY: IC1.20, JP4.2
- new net RST: JP3.1
- new net SIM_RX: IC1.17, JP3.3
- new net SIM_TX: IC1.16, JP3.4
- new net VDD: JP3.5
- new net VIN: C5.+, IC2.1, X2.1
- net 5V: now also C3.1, C4.2, C6.+, IC1.10, IC1.30, IC2.3, JP4.3, R1.1, T1.3; no longer X2.1
- net GND: now also C5.-, C6.-, IC2.2, JP1.1, JP1.3, JP1.5, JP2.2, JP3.2, JP4.1, X2.2; no longer LED1.K, LED2.K, LED3.K, X1.1
- net N$12: now also JP2.1; no longer X1.2
- net N$7: now also JP1.2; no longer LED1.A
- net N$8: now also JP1.4; no longer LED2.A
- net N$9: now also JP1.6; no longer LED3.A
