File: schema/mjBeep/boardBase.sch (EAGLE design)
At the start: 17 parts, among them IC1 atmega1284, Q1 16MH, T1 BC547

Commit message: mod
Parts:
- removed LED1, LED2, LED3: (no value), led:LED5MM
- removed X1: (no value), con-wago-500:W237-102
- added C5, C6: 100nF, rcl:CPOL-EUE3.5-10
- added IC2: 7805T, linear:7805T
- added JP1: LedPin, pinhead:PINHD-2X3
- added JP2: Spk, pinhead:PINHD-1X2
- added JP3: GSM, pinhead:PINHD-1X7
- added JP4: Relay, pinhead:PINHD-1X3
- R5: value (none) -> 230
- X2: value (none) -> VIN
Connections:
- net N$10 renamed SPK
- removed net N$14: X2-2.KL
- removed net N$4: IC1.T0/XCK0/PCINT8, R2.1
- removed net N$5: IC1.T1/CLK0/PCINT9, R3.1
- removed net N$6: IC1.AIN0/INT2/PCINT10, R4.1
- removed net VCC: C3.1, C4.2, IC1.AVCC, IC1.VCC, R1.1, T1.C
- new net GSM_5V: JP3.7
- new net GSM_GND: JP3.6
- new net LED_GIALLO: IC1.T1/CLK0/PCINT9, R2.1
- new net LED_ROSSO: IC1.AIN1/OC0A/PCINT11, R4.1
- new net LED_VERDE: IC1.AIN0/INT2/PCINT10, R3.1
- new net RELAY: IC1.OC2B/ICP/PCINT30, JP4.2
- new net RST: JP3.1
- new net SIM_RX: IC1.TXD1/INT1/PCINT27, JP3.3
- new net SIM_TX: IC1.RXD1/INT0/PCINT26, JP3.4
- new net VDD: JP3.5
- new net VIN: C5.+, IC2.VI, X2-1.KL
- net 5V: now also C3.1, C4.2, C6.+, IC1.AVCC, IC1.VCC, IC2.VO, JP4.3, R1.1, T1.C; no longer X2-1.KL
- net GND: now also C5.-, C6.-, IC2.GND, JP1.1, JP1.3, JP1.5, JP2.2, JP3.2, JP4.1, X2-2.KL; no longer LED1.C, LED2.C, LED3.C, X1-1.KL
- net N$12: now also JP2.1; no longer X1-2.KL
- net N$7: now also JP1.2; no longer LED1.A
- net N$8: now also JP1.4; no longer LED2.A
- net N$9: now also JP1.6; no longer LED3.A
Other:
- note added: "G.P.L. V3"
- note added: "GSM Modulo"
- note added: "LED"
- note added: "M&J - Beep"
- note added: "Power"
- note added: "Relay Sirena"
- note added: "Speaker"
- note added: "http://siatienfalla.altervista.org/"
- moved on the sheet: C1, C2, C3, C4, IC1, Q1, R1, R2, R3, R4, R5, T1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
