File: schema/mjBeep/boardBase3.brd (EAGLE design)
At the start: 92.4 x 73.7 mm, 57 parts, among them IC1 atmega1284, IC2 PCF8574P, IC3 PCF8574P, IC4 7805T, Q1 16MH, T1 BC547

Commit message: mod
Parts:
- removed IC3: PCF8574P, micro-philips:DIL16
- removed JP7: (no value), pinhead:2X03
- removed JP8: (no value), pinhead:1X16
- removed R11, R12, R13, R14, R15, R18, R19, R20, R21, R22, R23, R24, R25: 10K, rcl:0207/2V
- removed X1, X3: (no value), con-wago-508:W237-8P
- C6, C7: device rcl:E3,5-10 -> rcl:E2-4
- R10, R5, R6, R7, R8, R9: device rcl:0207/10 -> rcl:0207/2V
- moved C7 114.3 mm to (35.6, 55.9), turned to 270 degrees
- moved C6 93.6 mm to (35.6, 50.8), turned to 180 degrees
- moved IC4 62.9 mm to (16.5, 50.8), turned to 90 degrees
- moved H4 53.5 mm to (62.2, 8.89)
- moved H3 47.3 mm to (58.4, 48.3)
- moved PWR 38.6 mm to (24.1, 66.0), turned to 180 degrees
- moved SPK 28.8 mm to (53.3, 8.89), turned to 180 degrees
- moved T1 19.4 mm to (53.3, 17.8)
- moved R6 18.1 mm to (50.8, 55.9)
- moved R7 18.1 mm to (50.8, 53.3)
- moved R8 18.1 mm to (50.8, 58.4), turned to 0 degrees
- moved IC2 16.6 mm to (52.1, 66.0)
- moved JP3 16.6 mm to (44.5, 55.9)
- moved KEYPAD 15.3 mm to (64.8, 57.1)
- moved R9 14.9 mm to (36.8, 67.3)
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Connections:
- removed net N$10: IC2.14, R10.1
- removed net N$13: IC2.15, R9.1
- removed net N$14: IC3.1, JP7.2, R13.2
- removed net N$15: IC3.2, JP7.4, R11.2
- removed net N$16: IC3.3, JP7.6, R12.1
- removed net N$17: IC3.14, R15.1
- removed net N$18: IC3.15, R14.1
- removed net N$22: IC3.4, JP8.2, X1.8
- removed net N$23: IC3.5, JP8.4, X1.6
- removed net N$24: IC3.6, JP8.6, X1.4
- removed net N$25: IC3.7, JP8.8, X1.2
- removed net N$26: IC3.9, JP8.10, X3.8
- removed net N$27: IC3.10, JP8.12, X3.6
- removed net N$28: IC3.11, JP8.14, X3.4
- removed net N$29: IC3.12, JP8.16, X3.2
- removed net N$30: JP8.1, R18.2
- removed net N$31: JP8.3, R19.2
- removed net N$32: JP8.5, R20.2
- removed net N$33: JP8.7, R21.2
- removed net N$34: JP8.9, R22.2
- removed net N$35: JP8.11, R23.2
- removed net N$36: JP8.13, R24.2
- removed net N$37: JP8.15, R25.2
- removed net N$40: R20.1
- removed net VIN: C6.+, IC4.1
- new net 13V: C6.+, IC4.1, PWR.1
- net 5V: now also R10.1, R8.2, R9.2; no longer IC3.16, PWR.1, R11.1, R12.2, R13.1, R8.1, X1.1, X1.3, X1.5, X1.7, X3.1, X3.3, X3.5, X3.7
- net GND: no longer IC3.8, JP7.1, JP7.3, JP7.5, R18.1, R19.1, R21.1, R22.1, R23.1, R24.1, R25.1
- net N$3: now also R8.1; no longer R8.2
- net SCL: now also IC2.14; no longer R15.2
- net SDA: now also IC2.15, R9.1; no longer R14.2, R9.2
Routing:
- net GND: track 0.00 -> 196.8 mm
- net 5V: track 0.00 -> 148.5 mm
- net SDA: track 0.00 -> 47.8 mm
- net SCL: track 0.00 -> 46.5 mm
- net 13V: track 0.00 -> 30.8 mm
- net RESET: track 0.00 -> 24.8 mm
- net P0: track 0.00 -> 18.5 mm
- net P2: track 0.00 -> 17.9 mm
- net P7: track 0.00 -> 17.2 mm
- net N$4: track 0.00 -> 17.0 mm
- net RX: track 0.00 -> 16.8 mm
- net TX: track 0.00 -> 16.8 mm
- net P3: track 0.00 -> 16.6 mm
- net P1: track 0.00 -> 15.1 mm
- net N$6: track 0.00 -> 13.3 mm
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- added copper zone on layer 1, net N$10
- added copper zone on layer 16, net N$13
Other:
- board size 92.4 x 73.7 mm -> 63.2 x 69.8 mm
- board text added: "-"
- board text added: "13V"
- board text added: "2016"
- board text added: "mjBeep"

Commit message: mod
Parts:
- removed C6, C7: 100nF, rcl:E2-4
- removed IC4: 7805T, linear:TO220H
- removed LCD: LCD, pinhead:1X04
- removed RELAY: Relay, pinhead:1X03
- removed RTC: (no value), pinhead:1X04
- added I2C1: LCD, pinhead:1X04
- added I2C2, I2C3, I2C4, I2C5, I2C6: (no value), pinhead:1X04
- added REL1, REL2: Relay, pinhead:1X03
- moved PWR 42.6 mm to (62.2, 47.0), turned to 90 degrees
- moved JP3 35.8 mm to (10.2, 45.7)
- moved R7 35.8 mm to (16.5, 43.2)
- moved KEYPAD 35.7 mm to (29.2, 59.7), turned to 0 degrees
- moved R9 31.2 mm to (8.89, 53.3)
- moved R6 30.7 mm to (22.9, 43.2)
- moved IC2 29.6 mm to (26.7, 50.8)
- moved R8 26.4 mm to (29.2, 43.2)
- moved R10 26.2 mm to (14.0, 53.3), turned to 90 degrees
- moved H3 11.4 mm to (63.5, 58.4)
- moved H2 6.35 mm to (11.4, 59.7)
- moved C4 1.80 mm to (36.8, 43.2)
- moved H1 0.51 mm to (11.4, 8.13)
Connections:
- removed net 13V: C6.+, IC4.1, PWR.1
- removed net RELAY: IC1.20, RELAY.2
- new net RELAY1: IC1.20, REL1.2
- new net RELAY2: IC1.18, REL2.2
- net 5V: now also I2C1.1, I2C2.1, I2C3.1, I2C4.1, I2C5.1, I2C6.1, PWR.1, REL1.3, REL2.3; no longer C7.+, IC4.3, LCD.1, RELAY.3, RTC.1
- net GND: now also I2C1.2, I2C2.2, I2C3.2, I2C4.2, I2C5.2, I2C6.2, REL1.1, REL2.1; no longer C6.-, C7.-, IC4.2, LCD.2, RELAY.1, RTC.2
- net SCL: now also I2C1.4, I2C2.4, I2C3.4, I2C4.4, I2C5.4, I2C6.4; no longer LCD.4, RTC.4
- net SDA: now also I2C1.3, I2C2.3, I2C3.3, I2C4.3, I2C5.3, I2C6.3; no longer LCD.3, RTC.3
Routing:
- net 13V: track 30.8 -> 0.00 mm
- net SDA: track 47.8 -> 73.9 mm
- net SCL: track 46.5 -> 71.6 mm
- net 5V: track 148.5 -> 168.2 mm
- net P4: track 5.39 -> 21.8 mm
- net P7: track 17.2 -> 5.14 mm
- net N$3: track 8.79 -> 20.2 mm
- net RELAY2: track 0.00 -> 9.75 mm
- net GND: track 196.8 -> 204.8 mm
- net RELAY1: track 0.00 -> 7.91 mm
- net P5: track 8.98 -> 14.7 mm
- net RELAY: track 5.45 -> 0.00 mm
- net P6: track 12.6 -> 7.25 mm
- net P2: track 17.9 -> 14.8 mm
- net N$5: track 11.1 -> 14.0 mm
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Other:
- board size 63.2 x 69.8 mm -> 63.2 x 62.2 mm
- board text added: "5V"
- board text added: "GND"
- board text added: "SCL"
- board text added: "SDA"
- board text removed: "-"
- board text removed: "13V"

Commit message: mod
Parts:
- renumbered IC1 to ATMEGA1284
Changed lines of the file:
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@@
 <setting verticaltext="up"/>
 </settings>
-<grid distance="50" unitdist="mil" unit="mil" style="lines" multiple="1" display="no" altdistance="5" altunitdist="mil" altunit="mil"/>
+<grid distance="50" unitdist="mil" unit="mm" style="lines" multiple="1" display="no" altdistance="5" altunitdist="mil" altunit="mm"/>
 <layers>
 <layer number="1" name="Top" color="4" fill="1" visible="yes" active="yes"/>
@@
 <attribute name="VALUE" x="28.194" y="3.556" size="1.27" layer="27" ratio="10"/>
 </element>
-<element name="IC1" library="1284p" package="DIL40" value="atmega1284" x="36.83" y="31.75" smashed="yes">
+<element name="ATMEGA1284" library="1284p" package="DIL40" value="atmega1284" x="36.83" y="31.75" smashed="yes">
 <attribute name="NAME" x="26.416" y="30.988" size="1.778" layer="25"/>
 <attribute name="VALUE" x="19.685" y="30.734" size="1.778" layer="27"/>
@@
 <signals>
 <signal name="GND">
-<contactref element="IC1" pad="11"/>
-<contactref element="IC1" pad="31"/>
+<contactref element="ATMEGA1284" pad="11"/>
+<contactref element="ATMEGA1284" pad="31"/>
 <contactref element="C2" pad="1"/>
 <contactref element="C1" pad="1"/>
@@
 <signal name="N$1">
 <contactref element="Q1" pad="1"/>
-<contactref element="IC1" pad="12"/>
+<contactref element="ATMEGA1284" pad="12"/>
 <contactref element="C2" pad="2"/>
 <wire x1="40.775" y1="16.45" x2="40.775" y2="18.9" width="0.2" layer="1"/>
@@
 <signal name="N$2">
 <contactref element="Q1" pad="2"/>
-<contactref element="IC1" pad="13"/>
+<contactref element="ATMEGA1284" pad="13"/>
 <contactref element="C1" pad="2"/>
 <wire x1="45.675" y1="16.625" x2="45.675" y2="18.9" width="0.2" layer="1"/>
@@
 <signal name="SPK">
 <contactref element="R5" pad="1"/>
-<contactref element="IC1" pad="19"/>
+<contactref element="ATMEGA1284" pad="19"/>
 <wire x1="58.45" y1="23.975" x2="58.45" y2="20.475" width="0.2" layer="1"/>
 <wire x1="58.45" y1="20.475" x2="58.42" y2="20.32" width="0.2" layer="1"/>
@@
 </signal>
 <signal name="LED_GIALLO">
-<contactref element="IC1" pad="2"/>
+<contactref element="ATMEGA1284" pad="2"/>
 <contactref element="R2" pad="2"/>
 <wire x1="15.225" y1="23.975" x2="15.225" y2="21.7" width="0.2" layer="1"/>
@@
 <signal name="LED_VERDE">
 <contactref element="R3" pad="1"/>
-<contactref element="IC1" pad="3"/>
+<contactref element="ATMEGA1284" pad="3"/>
 <wire x1="17.85" y1="23.975" x2="17.85" y2="20.475" width="0.2" layer="1"/>
 <wire x1="17.85" y1="20.475" x2="17.78" y2="20.32" width="0.2" layer="1"/>
@@
 </signal>
 <signal name="LED_ROSSO">
-<contactref element="IC1" pad="4"/>
+<contactref element="ATMEGA1284" pad="4"/>
 <contactref element="R4" pad="2"/>
 <wire x1="20.3" y1="23.975" x2="20.3" y2="21.7" width="0.2" layer="1"/>
@@
 </signal>
 <signal name="5V">
-<contactref element="IC1" pad="10"/>
+<contactref element="ATMEGA1284" pad="10"/>
 <contactref element="C4" pad="2"/>
-<contactref element="IC1" pad="30"/>
+<contactref element="ATMEGA1284" pad="30"/>
 <contactref element="C3" pad="1"/>
 <contactref element="R1" pad="1"/>
@@
 </signal>
 <signal name="SIM_TX">
-<contactref element="IC1" pad="16"/>
+<contactref element="ATMEGA1284" pad="16"/>
 </signal>
 <signal name="SIM_RX">
-<contactref element="IC1" pad="17"/>
+<contactref element="ATMEGA1284" pad="17"/>
 </signal>
 <signal name="RESET">
 <contactref element="C5" pad="1"/>
-<contactref element="IC1" pad="9"/>
+<contactref element="ATMEGA1284" pad="9"/>
 <contactref element="R1" pad="2"/>
 <contactref element="S1" pad="3"/>
@@
 </signal>
 <signal name="TX">
-<contactref element="IC1" pad="15"/>
+<contactref element="ATMEGA1284" pad="15"/>
 <contactref element="FTDI" pad="2"/>
 <wire x1="44.45" y1="11.375" x2="44.45" y2="8.89" width="0.2" layer="1"/>
@@
 </signal>
 <signal name="RX">
-<contactref element="IC1" pad="14"/>
+<contactref element="ATMEGA1284" pad="14"/>
 <contactref element="FTDI" pad="3"/>
 <wire x1="42" y1="11.55" x2="42" y2="8.925" width="0.2" layer="16"/>
@@
 </signal>
 <signal name="SCL">
-<contactref element="IC1" pad="22"/>
+<contactref element="ATMEGA1284" pad="22"/>
 <contactref element="R10" pad="2"/>
 <contactref element="I2C1" pad="4"/>
@@
 </signal>
 <signal name="SDA">
-<contactref element="IC1" pad="23"/>
+<contactref element="ATMEGA1284" pad="23"/>
 <contactref element="R9" pad="1"/>
 <contactref element="I2C1" pad="3"/>
@@
 </signal>
 <signal name="LED_SIRENA">
-<contactref element="IC1" pad="5"/>
+<contactref element="ATMEGA1284" pad="5"/>
 <contactref element="R16" pad="1"/>
 <wire x1="22.925" y1="23.975" x2="22.925" y2="20.475" width="0.2" layer="1"/>
@@
 </signal>
 <signal name="N$20">
-<contactref element="IC1" pad="1"/>
+<contactref element="ATMEGA1284" pad="1"/>
 <contactref element="R17" pad="1"/>
 <wire x1="11.375" y1="24.15" x2="12.6" y2="24.15" width="0.2" layer="1"/>
@@
 </signal>
 <signal name="RELAY1">
-<contactref element="IC1" pad="20"/>
+<contactref element="ATMEGA1284" pad="20"/>
 <contactref element="REL1" pad="2"/>
 <wire x1="61.075" y1="21.525" x2="61.075" y2="23.975" width="0.2" layer="1"/>
@@
 </signal>
 <signal name="RELAY2">
-<contactref element="IC1" pad="18"/>
+<contactref element="ATMEGA1284" pad="18"/>
 <contactref element="REL2" pad="2"/>
 <wire x1="56.525" y1="24.15" x2="56" y2="24.15" width="0.2" layer="1"/>
