File: schema/mjBeep/boardBase3.sch (EAGLE design)
At the start: 57 parts, among them IC1 atmega1284, IC2 PCF8574P, IC3 PCF8574P, IC4 7805T, Q1 16MH, T1 BC547

Commit message: mod
Parts:
- removed IC3: PCF8574P, micro-philips:PCF8574P
- removed JP7: (no value), pinhead:PINHD-2X3
- removed JP8: (no value), pinhead:PINHD-1X16
- removed R11, R12, R13, R14, R15, R18, R19, R20, R21, R22, R23, R24, R25: 10K, rcl:R-EU_0207/2V
- removed X1, X3: (no value), con-wago-508:W237-08P
- C6, C7: device rcl:CPOL-EUE3.5-10 -> rcl:CPOL-EUE2-4
- R10, R5, R6, R7, R8, R9: device rcl:R-EU_0207/10 -> rcl:R-EU_0207/2V
Connections:
- removed net N$10: IC2.SCL, R10.1
- removed net N$13: IC2.SDA, R9.1
- removed net N$14: IC3.A0, JP7.2, R13.2
- removed net N$15: IC3.A1, JP7.4, R11.2
- removed net N$16: IC3.A2, JP7.6, R12.1
- removed net N$17: IC3.SCL, R15.1
- removed net N$18: IC3.SDA, R14.1
- removed net N$22: IC3.P0, JP8.2, X1-8.KL
- removed net N$23: IC3.P1, JP8.4, X1-6.KL
- removed net N$24: IC3.P2, JP8.6, X1-4.KL
- removed net N$25: IC3.P3, JP8.8, X1-2.KL
- removed net N$26: IC3.P4, JP8.10, X3-8.KL
- removed net N$27: IC3.P5, JP8.12, X3-6.KL
- removed net N$28: IC3.P6, JP8.14, X3-4.KL
- removed net N$29: IC3.P7, JP8.16, X3-2.KL
- removed net N$30: JP8.1, R18.2
- removed net N$31: JP8.3, R19.2
- removed net N$32: JP8.5, R20.2
- removed net N$33: JP8.7, R21.2
- removed net N$34: JP8.9, R22.2
- removed net N$35: JP8.11, R23.2
- removed net N$36: JP8.13, R24.2
- removed net N$37: JP8.15, R25.2
- removed net N$40: R20.1
- removed net VIN: C6.+, IC4.VI
- new net 13V: C6.+, IC4.VI, PWR-1.KL
- net 5V: now also R10.1, R8.2, R9.2; no longer IC3.VDD, PWR-1.KL, R11.1, R12.2, R13.1, R8.1, X1-1.KL, X1-3.KL, X1-5.KL, X1-7.KL, X3-1.KL, X3-3.KL, X3-5.KL, X3-7.KL
- net GND: no longer IC3.VSS, JP7.1, JP7.3, JP7.5, R18.1, R19.1, R21.1, R22.1, R23.1, R24.1, R25.1
- net N$3: now also R8.1; no longer R8.2
- net SCL: now also IC2.SCL; no longer R15.2
- net SDA: now also IC2.SDA, R9.1; no longer R14.2, R9.2
Other:
- note removed: "GND"
- moved on the sheet: C5, C6, C7, FTDI, H1, H4, IC4, LCD, LEDS, PWR-1, PWR-2, R10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

Commit message: mod
Parts:
- removed C6, C7: 100nF, rcl:CPOL-EUE2-4
- removed IC4: 7805T, linear:7805T
- added I2C3, I2C4, I2C5, I2C6: (no value), pinhead:PINHD-1X4
- added REL2: Relay, pinhead:PINHD-1X3
- renumbered LCD to I2C1, RELAY to REL1, RTC to I2C2
Connections:
- net RELAY renamed RELAY1
- removed net 13V: C6.+, IC4.VI, PWR-1.KL
- new net RELAY2: IC1.XCK1/OC1B/PCINT28, REL2.2
- net 5V: now also I2C3.1, I2C4.1, I2C5.1, I2C6.1, PWR-1.KL, REL2.3; no longer C7.+, IC4.VO
- net GND: now also I2C3.2, I2C4.2, I2C5.2, I2C6.2, REL2.1; no longer C6.-, C7.-, IC4.GND
- net SCL: now also I2C3.4, I2C4.4, I2C5.4, I2C6.4
- net SDA: now also I2C3.3, I2C4.3, I2C5.3, I2C6.3
Other:
- note removed: "Power"

Commit message: mod
Parts:
- renumbered IC1 to ATMEGA1284
Changed lines of the file:
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@@
 <setting verticaltext="up"/>
 </settings>
-<grid distance="0.1" unitdist="inch" unit="inch" style="lines" multiple="1" display="no" altdistance="0.01" altunitdist="inch" altunit="inch"/>
+<grid distance="0.1" unitdist="inch" unit="mm" style="lines" multiple="1" display="no" altdistance="0.01" altunitdist="inch" altunit="mm"/>
 <layers>
 <layer number="1" name="Top" color="4" fill="1" visible="no" active="no"/>
@@
 </classes>
 <parts>
-<part name="IC1" library="1284p" deviceset="MEGA1284P" device="" value="atmega1284"/>
+<part name="ATMEGA1284" library="1284p" deviceset="MEGA1284P" device="" value="atmega1284"/>
 <part name="Q1" library="special" deviceset="XTAL/S" device="" value="16MH"/>
 <part name="C1" library="rcl" deviceset="C-EU" device="025-024X044" value="22p"/>
@@
 </plain>
 <instances>
-<instance part="IC1" gate="G$1" x="27.94" y="40.64"/>
+<instance part="ATMEGA1284" gate="G$1" x="27.94" y="40.64"/>
 <instance part="Q1" gate="G$1" x="-10.16" y="33.02" smashed="yes" rot="R90">
 <attribute name="NAME" x="-13.97" y="30.48" size="1.778" layer="95" rot="R90"/>
@@
 <pinref part="SUPPLY1" gate="GND" pin="GND"/>
 <wire x1="-38.1" y1="25.4" x2="-38.1" y2="2.54" width="0.1524" layer="91"/>
-<pinref part="IC1" gate="G$1" pin="GND@1"/>
+<pinref part="ATMEGA1284" gate="G$1" pin="GND@1"/>
 <wire x1="-38.1" y1="2.54" x2="-38.1" y2="-2.54" width="0.1524" layer="91"/>
 <wire x1="-38.1" y1="-2.54" x2="5.08" y2="-2.54" width="0.1524" layer="91"/>
-<pinref part="IC1" gate="G$1" pin="GND@0"/>
+<pinref part="ATMEGA1284" gate="G$1" pin="GND@0"/>
 <wire x1="5.08" y1="2.54" x2="-38.1" y2="2.54" width="0.1524" layer="91"/>
 <pinref part="C2" gate="G$1" pin="1"/>
@@
 <segment>
 <pinref part="Q1" gate="G$1" pin="1"/>
-<pinref part="IC1" gate="G$1" pin="XTAL2"/>
+<pinref part="ATMEGA1284" gate="G$1" pin="XTAL2"/>
 <wire x1="-10.16" y1="27.94" x2="-5.08" y2="27.94" width="0.1524" layer="91"/>
 <pinref part="C2" gate="G$1" pin="2"/>
@@
 <segment>
 <pinref part="Q1" gate="G$1" pin="2"/>
-<pinref part="IC1" gate="G$1" pin="XTAL1"/>
+<pinref part="ATMEGA1284" gate="G$1" pin="XTAL1"/>
 <wire x1="-10.16" y1="38.1" x2="-5.08" y2="38.1" width="0.1524" layer="91"/>
 <pinref part="C1" gate="G$1" pin="2"/>
@@
 </segment>
 <segment>
-<pinref part="IC1" gate="G$1" pin="OC1A/PCINT29"/>
+<pinref part="ATMEGA1284" gate="G$1" pin="OC1A/PCINT29"/>
 <wire x1="50.8" y1="2.54" x2="60.96" y2="2.54" width="0.1524" layer="91"/>
 <label x="55.88" y="2.54" size="1.778" layer="95"/>
@@
 <net name="LED_GIALLO" class="0">
 <segment>
-<pinref part="IC1" gate="G$1" pin="T1/CLK0/PCINT9"/>
+<pinref part="ATMEGA1284" gate="G$1" pin="T1/CLK0/PCINT9"/>
 <wire x1="50.8" y1="58.42" x2="60.96" y2="58.42" width="0.1524" layer="91"/>
 <label x="55.88" y="58.42" size="1.778" layer="95"/>
@@
 </segment>
 <segment>
-<pinref part="IC1" gate="G$1" pin="AIN0/INT2/PCINT10"/>
+<pinref part="ATMEGA1284" gate="G$1" pin="AIN0/INT2/PCINT10"/>
 <wire x1="50.8" y1="55.88" x2="60.96" y2="55.88" width="0.1524" layer="91"/>
 <label x="55.88" y="55.88" size="1.778" layer="95"/>
@@
 <net name="LED_ROSSO" class="0">
 <segment>
-<pinref part="IC1" gate="G$1" pin="AIN1/OC0A/PCINT11"/>
+<pinref part="ATMEGA1284" gate="G$1" pin="AIN1/OC0A/PCINT11"/>
 <wire x1="50.8" y1="53.34" x2="60.96" y2="53.34" width="0.1524" layer="91"/>
 <label x="55.88" y="53.34" size="1.778" layer="95"/>
@@
 <net name="5V" class="0">
 <segment>
-<pinref part="IC1" gate="G$1" pin="VCC"/>
+<pinref part="ATMEGA1284" gate="G$1" pin="VCC"/>
 <wire x1="-25.4" y1="83.82" x2="5.08" y2="83.82" width="0.1524" layer="91"/>
 <pinref part="C4" gate="G$1" pin="2"/>
@@
 </segment>
 <segment>
-<pinref part="IC1" gate="G$1" pin="AVCC"/>
+<pinref part="ATMEGA1284" gate="G$1" pin="AVCC"/>
 <wire x1="5.08" y1="78.74" x2="-25.4" y2="78.74" width="0.1524" layer="91"/>
 <wire x1="-25.4" y1="78.74" x2="-38.1" y2="78.74" width="0.1524" layer="91"/>
@@
 <net name="SIM_TX" class="0">
 <segment>
-<pinref part="IC1" gate="G$1" pin="RXD1/INT0/PCINT26"/>
+<pinref part="ATMEGA1284" gate="G$1" pin="RXD1/INT0/PCINT26"/>
 <wire x1="50.8" y1="10.16" x2="60.96" y2="10.16" width="0.1524" layer="91"/>
 <label x="55.88" y="10.16" size="1.778" layer="95"/>
@@
 <net name="SIM_RX" class="0">
 <segment>
-<pinref part="IC1" gate="G$1" pin="TXD1/INT1/PCINT27"/>
+<pinref part="ATMEGA1284" gate="G$1" pin="TXD1/INT1/PCINT27"/>
 <wire x1="50.8" y1="7.62" x2="60.96" y2="7.62" width="0.1524" layer="91"/>
 <label x="55.88" y="7.62" size="1.778" layer="95"/>
@@
 </segment>
 <segment>
-<pinref part="IC1" gate="G$1" pin="RESET"/>
+<pinref part="ATMEGA1284" gate="G$1" pin="RESET"/>
 <pinref part="R1" gate="G$1" pin="2"/>
 <wire x1="5.08" y1="66.04" x2="0" y2="66.04" width="0.1524" layer="91"/>
@@
 <net name="TX" class="0">
 <segment>
-<pinref part="IC1" gate="G$1" pin="TXD0/PCINT25"/>
+<pinref part="ATMEGA1284" gate="G$1" pin="TXD0/PCINT25"/>
 <wire x1="50.8" y1="12.7" x2="60.96" y2="12.7" width="0.1524" layer="91"/>
 <label x="55.88" y="12.7" size="1.778" layer="95"/>
@@
 <net name="RX" class="0">
 <segment>
-<pinref part="IC1" gate="G$1" pin="T3/RXD0/PCINT24"/>
+<pinref part="ATMEGA1284" gate="G$1" pin="T3/RXD0/PCINT24"/>
 <wire x1="50.8" y1="15.24" x2="60.96" y2="15.24" width="0.1524" layer="91"/>
 <label x="55.88" y="15.24" size="1.778" layer="95"/>
@@
 <net name="SCL" class="0">
 <segment>
-<pinref part="IC1" gate="G$1" pin="SCL/PCINT16"/>
+<pinref part="ATMEGA1284" gate="G$1" pin="SCL/PCINT16"/>
 <wire x1="50.8" y1="38.1" x2="63.5" y2="38.1" width="0.1524" layer="91"/>
 <label x="58.42" y="38.1" size="1.778" layer="95"/>
@@
 <net name="SDA" class="0">
 <segment>
-<pinref part="IC1" gate="G$1" pin="SDA/PCINT17"/>
+<pinref part="ATMEGA1284" gate="G$1" pin="SDA/PCINT17"/>
 <wire x1="50.8" y1="35.56" x2="63.5" y2="35.56" width="0.1524" layer="91"/>
 <label x="58.42" y="35.56" size="1.778" layer="95"/>
@@
 <net name="LED_SIRENA" class="0">
 <segment>
-<pinref part="IC1" gate="G$1" pin="SS/OC0B/PCINT12"/>
+<pinref part="ATMEGA1284" gate="G$1" pin="SS/OC0B/PCINT12"/>
 <wire x1="50.8" y1="50.8" x2="60.96" y2="50.8" width="0.1524" layer="91"/>
 <label x="55.88" y="50.8" size="1.778" layer="95"/>
@@
 <net name="N$20" class="0">
 <segment>
-<pinref part="IC1" gate="G$1" pin="T0/XCK0/PCINT8"/>
+<pinref part="ATMEGA1284" gate="G$1" pin="T0/XCK0/PCINT8"/>
 <pinref part="R17" gate="G$1" pin="1"/>
 <wire x1="50.8" y1="60.96" x2="55.88" y2="60.96" width="0.1524" layer="91"/>
@@
 <net name="RELAY1" class="0">
 <segment>
-<pinref part="IC1" gate="G$1" pin="OC2B/ICP/PCINT30"/>
+<pinref part="ATMEGA1284" gate="G$1" pin="OC2B/ICP/PCINT30"/>
 <wire x1="50.8" y1="0" x2="60.96" y2="0" width="0.1524" layer="91"/>
 <label x="55.88" y="0" size="1.778" layer="95"/>
@@
 <net name="RELAY2" class="0">
 <segment>
-<pinref part="IC1" gate="G$1" pin="XCK1/OC1B/PCINT28"/>
+<pinref part="ATMEGA1284" gate="G$1" pin="XCK1/OC1B/PCINT28"/>
 <wire x1="50.8" y1="5.08" x2="60.96" y2="5.08" width="0.1524" layer="91"/>
 <label x="55.88" y="5.08" size="1.778" layer="95"/>
