File: schema/mjBeep/schedaSensori.brd (EAGLE design)
At the start: 60.6 x 41.9 mm, 22 parts, among them IC3 PCF8574P

Commit message: mod
Parts:
- moved H4 4.58 mm to (47.0, 14.0)
Routing:
- net N$29: track 64.7 -> 65.5 mm
Other:
- board text added: "5V"
- board text added: "GND"
- board text added: "SCL"
- board text added: "SDA"
Changed lines of the file:
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@@
 <setting verticaltext="up"/>
 </settings>
-<grid distance="50" unitdist="mil" unit="mil" style="lines" multiple="1" display="no" altdistance="5" altunitdist="mil" altunit="mil"/>
+<grid distance="50" unitdist="mil" unit="mm" style="lines" multiple="1" display="no" altdistance="5" altunitdist="mil" altunit="mm"/>
 <layers>
 <layer number="1" name="Top" color="4" fill="1" visible="yes" active="yes"/>
@@
 <text x="31.75" y="36.83" size="1.778" layer="1">mjSens</text>
 <text x="31.75" y="36.83" size="1.778" layer="16">mjSens</text>
+<text x="25.56" y="40" size="0.4064" layer="1" rot="R90">SDA</text>
+<text x="28.04" y="40" size="0.4064" layer="1" rot="R90">SCL</text>
+<text x="23.1" y="40.7" size="0.4064" layer="1" rot="R90">5V</text>
+<text x="20.53" y="40.7" size="0.3048" layer="1" rot="R90">GND</text>
 </plain>
 <attributes>
@@
 </class>
 </classes>
-<designrules name="eC_2Layer_PClass6_BaseCopperO18_eCDefault *">
+<designrules name="schedaSensori">
 <description language="de">
 &lt;p&gt;
@@
 <param name="mtIsolate" value="1.55mm 0.71mm 0.36mm 0.2mm 0.2mm 0.2mm 0.2mm 0.15mm 0.2mm 0.15mm 0.2mm 0.15mm 0.2mm 0.15mm 0.2mm"/>
 <param name="mdWireWire" value="0.25mm"/>
-<param name="mdWirePad" value="0.2mm"/>
-<param name="mdWireVia" value="0.2mm"/>
-<param name="mdPadPad" value="0.15mm"/>
-<param name="mdPadVia" value="0.15mm"/>
-<param name="mdViaVia" value="0.15mm"/>
+<param name="mdWirePad" value="0.205mm"/>
+<param name="mdWireVia" value="0.205mm"/>
+<param name="mdPadPad" value="0.205mm"/>
+<param name="mdPadVia" value="0.205mm"/>
+<param name="mdViaVia" value="0.205mm"/>
 <param name="mdSmdPad" value="0mil"/>
 <param name="mdSmdVia" value="0mil"/>
@@
 <element name="H2" library="holes" library_urn="urn:adsk.eagle:library:237" package="3,2" package3d_urn="urn:adsk.eagle:package:14275/1" value="MOUNT-HOLE3.2" x="5.08" y="5.08" smashed="yes"/>
 <element name="H3" library="holes" library_urn="urn:adsk.eagle:library:237" package="3,2" package3d_urn="urn:adsk.eagle:package:14275/1" value="MOUNT-HOLE3.2" x="45.72" y="36.83" smashed="yes"/>
-<element name="H4" library="holes" library_urn="urn:adsk.eagle:library:237" package="3,2" package3d_urn="urn:adsk.eagle:package:14275/1" value="MOUNT-HOLE3.2" x="44.45" y="17.78" smashed="yes"/>
+<element name="H4" library="holes" library_urn="urn:adsk.eagle:library:237" package="3,2" package3d_urn="urn:adsk.eagle:package:14275/1" value="MOUNT-HOLE3.2" x="46.99" y="13.97" smashed="yes"/>
 <element name="IC3" library="micro-philips" package="DIL16" value="PCF8574P" x="27.94" y="29.21" smashed="yes">
 <attribute name="MF" value="" x="27.94" y="29.21" size="1.778" layer="27" display="off"/>
@@
 <wire x1="29.425" y1="33.275" x2="29.21" y2="33.02" width="0.3" layer="1"/>
 <wire x1="55" y1="33.55" x2="55.245" y2="33.782" width="0.3" layer="1"/>
-<wire x1="45.375" y1="11.55" x2="36.85" y2="11.55" width="0.3" layer="1"/>
-<wire x1="56.1" y1="22.275" x2="45.375" y2="11.55" width="0.3" layer="1"/>
-<wire x1="56.65" y1="22.275" x2="56.1" y2="22.275" width="0.3" layer="1"/>
+<wire x1="37.755" y1="16.63" x2="36.85" y2="11.55" width="0.3" layer="1"/>
+<wire x1="54.83" y1="21.005" x2="37.755" y2="16.63" width="0.3" layer="1"/>
+<wire x1="56.65" y1="22.275" x2="54.83" y2="21.005" width="0.3" layer="1"/>
 <wire x1="57.475" y1="23.1" x2="56.65" y2="22.275" width="0.3" layer="1"/>
 <wire x1="57.475" y1="29.425" x2="57.475" y2="23.1" width="0.3" layer="1"/>
