File: schema/mjBeep/schedaSensori.sch (EAGLE design)
At the start: 22 parts, among them IC3 PCF8574P

Commit message: mod
Parts:
- removed JP8: (no value), pinhead:PINHD-1X16
- added JP1: (no value), pinhead:PINHD-1X4
- R11, R12, R13, R14, R15, R18, R19, R20, R21, R22, R23, R24, R25: device rcl:R-EU_0207/2V -> rcl:R-EU_0207/10
Connections:
- removed net N$30: JP8.1, R18.2
- removed net N$31: JP8.3, R19.2
- removed net N$32: JP8.5, R20.2
- removed net N$33: JP8.7, R21.2
- removed net N$34: JP8.9, R22.2
- removed net N$35: JP8.11, R23.2
- removed net N$36: JP8.13, R24.2
- removed net N$37: JP8.15, R25.2
- removed net N$40: R20.1
- net 5V: now also JP1.3
- net GND: now also JP1.4, R20.1
- net N$22: now also R18.2; no longer JP8.2
- net N$23: now also R19.2; no longer JP8.4
- net N$24: now also R20.2; no longer JP8.6
- net N$25: now also R21.2; no longer JP8.8
- net N$26: now also R22.2; no longer JP8.10
- net N$27: now also R23.2; no longer JP8.12
- net N$28: now also R24.2; no longer JP8.14
- net N$29: now also R25.2; no longer JP8.16
- net SCL: now also JP1.1
- net SDA: now also JP1.2
Other:
- note removed: "GND"
- moved on the sheet: H1, H2, H3, H4
